File: amplificador_200w.kicad_pcb (KiCad board)
At the start: 2 copper layers, 81 x 56 mm, 42 parts, among them J1 Conn_01x03, J2 Conn_01x03, J3 Conn_01x02, Q1 A733, Q2 A733, Q3 2SC2229, Q4 2SC2229, Q5 TIP42, Q6 TIP41, Q7 TIP42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

Commit message: enviando a fabricar a jlcpcb
Parts:
- removed G***: LOGO, MSS_Devices:logo-mr_solder_7.8x3.6mm
- RV1: value 1K -> 200
- moved RV1 121.9 mm to (142.9, 114.1), turned to -90 degrees
- moved C5 118.1 mm to (134.5, 114.7)
- moved C4 118.1 mm to (134.5, 106.2)
- moved C3 117.5 mm to (130.3, 96.1)
- moved D2 117.5 mm to (137.3, 99.1)
- moved Q3 117.5 mm to (130.3, 109.9)
- moved Q4 117.5 mm to (129.3, 113.3)
- moved R13 117.5 mm to (158.3, 94.3)
- moved R14 117.5 mm to (158.3, 118.9)
- moved C1 117.5 mm to (109.9, 98.7)
- moved C2 117.5 mm to (116.3, 87.5)
- moved C7 117.5 mm to (143.5, 121.9)
- moved D1 117.5 mm to (112.9, 93.9)
- moved D3 117.5 mm to (147.5, 104.0)
- moved H1 117.5 mm to (107.0, 75.0)
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Connections:
- net Net-(C5-Pad1) renamed /CC
Routing:
- net /CC: track 45.0 -> 2.80 mm
- net -50V: track 80.6 -> 85.6 mm
- net 50V: track 128.4 -> 130.9 mm
- net Net-(Q6-E): track 16.1 -> 18.0 mm
- net Net-(D3-A): track 38.4 -> 36.8 mm
- net Net-(D4-K): track 5.33 -> 3.90 mm
- net Net-(Q2-C): track 26.3 -> 24.9 mm
- net Net-(Q3-C): track 9.68 -> 10.6 mm
- net Net-(J3-Pin_1): track 107.7 -> 106.9 mm
- net Net-(Q1-C): track 31.0 -> 31.7 mm
- added copper zone on B.Cu, net /CC
Other:
- board text added: "0"
- board text added: "0 mm"
- board text added: "0.01 mm"
- board text added: "0.02"
- board text added: "0.035 mm"
- board text added: "0.2000 mm / 0.0000 mm"
- board text added: "0.3000 mm"
- board text added: "1"
- board text added: "1.51 mm"
- board text added: "1.6000 mm"
- board text added: "2"
- board text added: "3.3"
- board text added: "4.5"
- board text added: "81.0000 mm x 56.0000 mm"
- board text added: "B.Cu"
- board text added: "B.Mask"
- board text added: "B.Paste"
- board text added: "B.Silkscreen"
- board text added: "BOARD CHARACTERISTICS"
- board text added: "Board Thickness:"
- board text added: "Board overall dimensions:"
- board text added: "Bottom Silk Screen"
- board text added: "Bottom Solder Mask"
- board text added: "Bottom Solder Paste"
- board text added: "Castellated pads:"
- board text added: "Color"
- board text added: "Copper Finish:"
- board text added: "Copper Layer Count:"
- board text added: "Dielectric 1"
- board text added: "Direct Printing"
- board text added: "Edge card connectors:"
- board text added: "Epsilon R"
- board text added: "F.Cu"
- board text added: "F.Mask"
- board text added: "F.Paste"
- board text added: "F.Silkscreen"
- board text added: "FR4"
- board text added: "FR4 natural"
- board text added: "Green"
- board text added: "HAL SnPb"
- board text added: "Impedance Control:"
- board text added: "Layer Name"
- board text added: "Liquid Ink"
- board text added: "Loss Tangent"
- board text added: "Material"
- board text added: "MaykolRey.com 2024"
- board text added: "Min hole diameter:"
- board text added: "Min track/spacing:"
- board text added: "No"
- board text added: "Plated Board Edge:"
- board text added: "Thickness (mm)"
- board text added: "Top Silk Screen"
- board text added: "Top Solder Mask"
- board text added: "Top Solder Paste"
- board text added: "Type"
- board text added: "White"
- board text added: "copper"
- board text added: "core"

Commit message: version simulada y probada en la realidad
Parts:
- C2: value 100uF -> 100u
- C7: value 10nF -> 10n
- R1: value 68K -> 68k
- R2, R5: value 3.3K -> 3.3k
- R3: value 4.7K -> 4.7k
- R4: value 33K -> 33k
- R6: value 1K -> 1k
- R7: value 68K -> 15k
Connections:
- net 50V renamed 27V
- net Net-(J1-Pin_2) renamed /input
- net Net-(J3-Pin_1) renamed /output
- R10 pad 1: -50V -> -27V
- R14 pad 1: -50V -> -27V
- R16 pad 1: -50V -> -27V
- R2 pad 2: -50V -> -27V
- R5 pad 2: -50V -> -27V
Routing:
- net -50V: track 85.6 -> 0.00 mm
- net -27V: track 0.00 -> 85.6 mm
