File: amplificador_200w.kicad_sch (KiCad schematic)
At the start: 41 parts, among them J1 Conn_01x03, J2 Conn_01x03, J3 Conn_01x02, Q1 A733, Q2 A733, Q3 2SC2229, Q4 2SC2229, Q5 TIP42, Q6 TIP41, Q7 TIP42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

Commit message: enviando a fabricar a jlcpcb
Connections:
- net CC: now reaches C5.1, C7.1, Q4.2 (C), Q7.1 (B), RV1.2, RV1.3

Commit message: version simulada y probada en la realidad
Parts:
- removed RV1: 200, Potentiometer_THT:Potentiometer_Runtron_RM-065_Vertical, symbol Device:R_Potentiometer
- added R12: 8, Resistor_THT:R_Axial_Power_L25.0mm_W9.0mm_P10.16mm_Vertical, symbol Device:R_US
- added RV1: 100, symbol Device:R_Potentiometer_US
- added V1, V2: 27, symbol Simulation_SPICE:VDC
- added V3: VSIN, symbol Simulation_SPICE:VSIN
- C2: value 100uF -> 100u
- C7: value 10nF -> 10n
- R1: value 68K -> 68k; symbol Device:R -> Device:R_US
- R10, R11, R13, R14, R15, R16, R8, R9: symbol Device:R -> Device:R_US
- R2, R5: value 3.3K -> 3.3k; symbol Device:R -> Device:R_US
- R3: value 4.7K -> 4.7k; symbol Device:R -> Device:R_US
- R4: value 33K -> 33k; symbol Device:R -> Device:R_US
- R6: value 1K -> 1k; symbol Device:R -> Device:R_US
- R7: value 68K -> 15k; symbol Device:R -> Device:R_US
Connections:
- net -50V: no longer R10.1, R14.1, R16.1, R2.2, R5.2
- net 50V: no longer C6.2, Q6.2 (C), Q8.2 (C), R11.2, R3.1, R8.2
- net CC: now also RV1.2
- net GND: now also R12.1, V1.2, V2.1, V3.2
- net input: now reaches C1.2, J1.2 (Pin_2)
- net input: now also V3.1
- net output: now reaches J3.1 (Pin_1), Q7.3 (E), Q9.2 (C), R13.1, R15.1, R7.1
- net output: now also R12.2
- net at D4.1 (K): now also RV1.1
- new net -27V: R10.1, R14.1, R16.1, R2.2, R5.2, V2.2
- new net 27V: C6.2, Q6.2 (C), Q8.2 (C), R11.2, R3.1, R8.2, V1.1
- no-connect marks 0 -> 1
Other:
- note added: "For Simulation"
- moved on the sheet: C1, C2, C3, C4, C5, C6, C7, D1, D3, J1, J2, J3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
