File: Simulations/amplificador_200w.kicad_sch (KiCad schematic)
At the start: 39 parts, among them Q1 A733, Q2 A733, Q3 2SC2229, Q4 2SC2229, Q5 TIP42, Q6 TIP41, Q7 TIP42, Q8 2SC5200, Q9 2SC5200

Commit message: version simulada y probada en la realidad
Parts:
- D1: Spice_Lib_File /home/maykol/Documentos/spice/kdzvtf24b.lib -> (none); Spice_Model DKDZVTF24B -> (none); Spice_Netlist_Enabled Y -> (none); Spice_Node_Sequence 2 1 -> (none); Spice_Primitive D -> (none)
- D2, D3, D4: Spice_Lib_File /home/maykol/Documentos/spice/2n3906.mod -> (none); Spice_Model 1N4007 -> (none); Spice_Netlist_Enabled Y -> (none); Spice_Node_Sequence 2 1 -> (none); Spice_Primitive D -> (none)
- Q1, Q2: Spice_Lib_File /home/maykol/Documentos/spice/2n3906.mod -> (none); Spice_Model KSA733 -> (none); Spice_Netlist_Enabled Y -> (none); Spice_Node_Sequence 2 3 1 -> (none); Spice_Primitive Q -> (none)
- Q3, Q4: Spice_Lib_File /home/maykol/Documentos/spice/2n3906.mod -> (none); Spice_Model 2SC2229 -> (none); Spice_Netlist_Enabled Y -> (none); Spice_Node_Sequence 2 3 1 -> (none); Spice_Primitive Q -> (none)
- Q5: Spice_Lib_File /home/maykol/Documentos/spice/2n5401.lib -> (none); Spice_Model 2N5401 -> (none); Spice_Netlist_Enabled Y -> (none); Spice_Node_Sequence 2 1 3 -> (none); Spice_Primitive Q -> (none)
- Q6, Q7: Spice_Lib_File /home/maykol/Documentos/spice/2n5551.lib -> (none); Spice_Model 2N5551 -> (none); Spice_Netlist_Enabled Y -> (none); Spice_Node_Sequence 2 1 3 -> (none); Spice_Primitive Q -> (none)
- Q8, Q9: Spice_Lib_File /home/maykol/Documentos/spice/2SC5200.mod -> (none); Spice_Model 2SC5200 -> (none); Spice_Netlist_Enabled Y -> (none); Spice_Node_Sequence 2 1 3 -> (none); Spice_Primitive Q -> (none)
- V1, V2: value VDC -> 50; Spice_Model dc 50 -> (none); Spice_Netlist_Enabled Y -> (none); Spice_Primitive V -> (none)
- V3: Spice_Model dc 1 ac 1 sin(0 1 1k) -> (none); Spice_Netlist_Enabled Y -> (none); Spice_Primitive V -> (none)
